File: PCB/grabert.kicad_pcb (KiCad board)
At the start: 2 copper layers, 285.8 x 120.7 mm, 14 parts, among them J1 Conn_01x02, J2 Conn_01x02, J3 Conn_01x05, J4 USB_C_Receptacle_USB2.0, J5 SSD1306, SW1 RotaryEncoder_Switch, U1 AMS1117-3.3, U2 STM32F072V8Tx

Commit message: switches placed
Parts:
- added SW0_0: 1.00u, kobuss-footprint:MX_1u, F.Cu at (9.53, -85.7)
- added SW0_1: 1.00u, kobuss-footprint:MX_1u, F.Cu at (28.6, -85.7)
- added SW0_10: 1.00u, kobuss-footprint:MX_1u, F.Cu at (200.0, -85.7)
- added SW0_11: 1.00u, kobuss-footprint:MX_1u, F.Cu at (219.1, -85.7)
- added SW0_12: 1.00u, kobuss-footprint:MX_1u, F.Cu at (238.1, -85.7)
- added SW0_13-14: 2.00u_or_1.00and1.00, kobuss-footprint:MX_2.00u_or_1.00and1.00, F.Cu at (266.7, -85.7)
- added SW0_2: 1.00u, kobuss-footprint:MX_1u, F.Cu at (47.6, -85.7)
- added SW0_3: 1.00u, kobuss-footprint:MX_1u, F.Cu at (66.7, -85.7)
- added SW0_4: 1.00u, kobuss-footprint:MX_1u, F.Cu at (85.7, -85.7)
- added SW0_5: 1.00u, kobuss-footprint:MX_1u, F.Cu at (104.8, -85.7)
- added SW0_6: 1.00u, kobuss-footprint:MX_1u, F.Cu at (123.8, -85.7)
- added SW0_7: 1.00u, kobuss-footprint:MX_1u, F.Cu at (142.9, -85.7)
- added SW0_8: 1.00u, kobuss-footprint:MX_1u, F.Cu at (161.9, -85.7)
- added SW0_9: 1.00u, kobuss-footprint:MX_1u, F.Cu at (181.0, -85.7)
- added SW1_0: 1.50u, kobuss-footprint:MX_1.50u, F.Cu at (14.3, -66.7)
- added SW1_1: 1.00u, kobuss-footprint:MX_1u, F.Cu at (38.1, -66.7)
- added SW1_10: 1.00u, kobuss-footprint:MX_1u, F.Cu at (209.6, -66.7)
- added SW1_11: 1.00u, kobuss-footprint:MX_1u, F.Cu at (228.6, -66.7)
- added SW1_12: 1.00u, kobuss-footprint:MX_1u, F.Cu at (247.7, -66.7)
- added SW1_13: 1.50u, kobuss-footprint:MX_1.50u, F.Cu at (271.5, -66.7)
- added SW1_2: 1.00u, kobuss-footprint:MX_1u, F.Cu at (57.1, -66.7)
- added SW1_3: 1.00u, kobuss-footprint:MX_1u, F.Cu at (76.2, -66.7)
- added SW1_4: 1.00u, kobuss-footprint:MX_1u, F.Cu at (95.2, -66.7)
- added SW1_5: 1.00u, kobuss-footprint:MX_1u, F.Cu at (114.3, -66.7)
- added SW1_6: 1.00u, kobuss-footprint:MX_1u, F.Cu at (133.3, -66.7)
- added SW1_7: 1.00u, kobuss-footprint:MX_1u, F.Cu at (152.4, -66.7)
- added SW1_8: 1.00u, kobuss-footprint:MX_1u, F.Cu at (171.4, -66.7)
- added SW1_9: 1.00u, kobuss-footprint:MX_1u, F.Cu at (190.5, -66.7)
- added SW2_0: 1.75u_stepped_caps_lock, kobuss-footprint:MX_1.75u_stepped_caps, F.Cu at (16.7, -47.6)
- added SW2_1: 1.00u, kobuss-footprint:MX_1u, F.Cu at (42.9, -47.6)
- added SW2_10: 1.00u, kobuss-footprint:MX_1u, F.Cu at (214.3, -47.6)
- added SW2_11: 1.00u, kobuss-footprint:MX_1u, F.Cu at (233.4, -47.6)
- added SW2_12: 2.25u, kobuss-footprint:MX_2.25u, F.Cu at (264.3, -47.6)
- added SW2_2: 1.00u, kobuss-footprint:MX_1u, F.Cu at (61.9, -47.6)
- added SW2_3: 1.00u, kobuss-footprint:MX_1u, F.Cu at (81.0, -47.6)
- added SW2_4: 1.00u, kobuss-footprint:MX_1u, F.Cu at (100.0, -47.6)
- added SW2_5: 1.00u, kobuss-footprint:MX_1u, F.Cu at (119.1, -47.6)
- added SW2_6: 1.00u, kobuss-footprint:MX_1u, F.Cu at (138.1, -47.6)
- added SW2_7: 1.00u, kobuss-footprint:MX_1u, F.Cu at (157.2, -47.6)
- added SW2_8: 1.00u, kobuss-footprint:MX_1u, F.Cu at (176.2, -47.6)
- added SW2_9: 1.00u, kobuss-footprint:MX_1u, F.Cu at (195.3, -47.6)
- added SW3_0-1: 2.25u_or_1.25and1.00, kobuss-footprint:MX_2.25u_or_1.25and1.00, F.Cu at (21.4, -28.6)
- added SW3_10: 1.00u, kobuss-footprint:MX_1u, F.Cu at (204.8, -28.6)
- added SW3_11: 1.00u, kobuss-footprint:MX_1u, F.Cu at (223.8, -28.6)
- added SW3_12-13: 2.75u_or_1.75and1.00, kobuss-footprint:MX_2.75u_or_1.75and1.00, F.Cu at (259.6, -28.6)
- added SW3_2: 1.00u, kobuss-footprint:MX_1u, F.Cu at (52.4, -28.6)
- added SW3_3: 1.00u, kobuss-footprint:MX_1u, F.Cu at (71.4, -28.6)
- added SW3_4: 1.00u, kobuss-footprint:MX_1u, F.Cu at (90.5, -28.6)
- added SW3_5: 1.00u, kobuss-footprint:MX_1u, F.Cu at (109.5, -28.6)
- added SW3_6: 1.00u, kobuss-footprint:MX_1u, F.Cu at (128.6, -28.6)
- added SW3_7: 1.00u, kobuss-footprint:MX_1u, F.Cu at (147.6, -28.6)
- added SW3_8: 1.00u, kobuss-footprint:MX_1u, F.Cu at (166.7, -28.6)
- added SW3_9: 1.00u, kobuss-footprint:MX_1u, F.Cu at (185.7, -28.6)
- added SW4_0: 1.25u, kobuss-footprint:MX_1.25, F.Cu at (11.9, -9.53)
- added SW4_1: 1.25u, kobuss-footprint:MX_1.25, F.Cu at (35.7, -9.53)
- added SW4_2: 1.25u, kobuss-footprint:MX_1.25, F.Cu at (59.5, -9.53)
- added SW4_3: 6.25u, kobuss-footprint:MX_6.25u, F.Cu at (131.0, -9.53)
- added SW4_4-8: 4x1.25u_or_5x1.00u, kobuss-footprint:MX_4x1.25u_or_5x1.00u, F.Cu at (238.1, -9.53)
- moved SW1 265.0 mm to (262.9, -110.5)
- moved R4 245.9 mm to (240.5, -104.3)
- moved C2 244.8 mm to (253.7, -114.4)
- moved R3 233.2 mm to (227.4, -111.9)
- moved C1 219.5 mm to (236.7, -115.7)
- moved J4 219.5 mm to (240.0, -110.5)
- moved U1 219.5 mm to (250.3, -107.6)
- moved U2 109.1 mm to (138.4, -108.0)
- moved R2 106.4 mm to (34.3, -114.3)
- moved J1 105.6 mm to (33.0, -118.1), turned to 90 degrees
- moved R1 103.1 mm to (24.1, -113.0)
- moved J2 102.6 mm to (21.6, -118.1), turned to 90 degrees
- moved J3 91.8 mm to (49.5, -116.8), turned to 90 degrees
- moved J5 73.7 mm to (9.84, -115.3)

Commit message: fixed component positions
Parts:
- moved U1 24.3 mm to (227.3, -115.6), turned to 180 degrees
- moved C2 20.0 mm to (233.7, -114.3), turned to -90 degrees
- moved R3 19.7 mm to (246.4, -106.7)
- moved R1 17.3 mm to (7.62, -118.1), turned to 180 degrees
- moved R2 14.5 mm to (20.3, -118.1)
- moved J3 14.0 mm to (35.6, -118.1)
- moved SW1 10.1 mm to (252.8, -111.7)
- moved J2 8.89 mm to (12.7, -118.1)
- moved J1 5.08 mm to (27.9, -118.1), turned to -90 degrees
- moved U2 4.44 mm to (142.9, -108.0), turned to 45 degrees
- moved J4 4.44 mm to (243.8, -112.8), turned to 180 degrees
- moved R4 2.52 mm to (241.3, -106.7), turned to 180 degrees
- moved J5 1.56 mm to (8.46, -114.6)
- moved C1 1.49 mm to (236.2, -114.3), turned to -90 degrees
