File: PCB/grabert.kicad_pcb (KiCad board)
At the start: 2 copper layers, 285.8 x 120.7 mm, 72 parts, among them J1 Conn_01x02, J2 Conn_01x02, J3 Conn_01x05, J4 USB_C_Receptacle_USB2.0, J5 SSD1306, SW0_0 1.00u, SW0_1 1.00u, SW0_10 1.00u, SW0_11 1.00u, SW0_12 1.00u, SW0_13-14 2.00u_or_1.00and1.00, SW0_2 1.00u, SW0_3 1.00u, SW0_4 1.00u, SW0_5 1.00u, SW0_6 1.00u, SW0_7 1.00u, SW0_8 1.00u, SW0_9 1.00u, SW1 RotaryEncoder_Switch, SW1_0 1.50u, SW1_1 1.00u, SW1_10 1.00u, SW1_11 1.00u, SW1_12 1.00u, SW1_13 1.50u, SW1_2 1.00u, SW1_3 1.00u, SW1_4 1.00u, SW1_5 1.00u, SW1_6 1.00u, SW1_7 1.00u, SW1_8 1.00u, SW1_9 1.00u, SW2_0 1.75u_stepped_caps_lock, SW2_1 1.00u, SW2_10 1.00u, SW2_11 1.00u, SW2_12 2.25u, SW2_2 1.00u, SW2_3 1.00u, SW2_4 1.00u, SW2_5 1.00u, SW2_6 1.00u, SW2_7 1.00u, SW2_8 1.00u, SW2_9 1.00u, SW3_0-1 2.25u_or_1.25and1.00, SW3_10 1.00u, SW3_11 1.00u, SW3_12-13 2.75u_or_1.75and1.00, SW3_2 1.00u, SW3_3 1.00u, SW3_4 1.00u, SW3_5 1.00u, SW3_6 1.00u, SW3_7 1.00u, SW3_8 1.00u, SW3_9 1.00u, SW4_0 1.25u, SW4_1 1.25u, SW4_2 1.25u, SW4_3 6.25u, SW4_4-8 4x1.25u_or_5x1.00u, U1 AMS1117-3.3, U2 STM32F072V8Tx

Commit message: Switch inputs linked to mcu
Connections:
- J5 pad 6: (no net) -> Net-(J5-Pad6)
- U2 pad 1: Net-(U2-Pad1) -> K3_2
- U2 pad 10: Net-(U2-Pad10) -> K2_3
- U2 pad 11: Net-(U2-Pad11) -> K1_4
- U2 pad 15: Net-(U2-Pad15) -> K0_5
- U2 pad 16: Net-(U2-Pad16) -> K3_4
- U2 pad 17: Net-(U2-Pad17) -> K2_4
- U2 pad 18: Net-(U2-Pad18) -> K1_5
- U2 pad 19: Net-(U2-Pad19) -> K0_6
- U2 pad 2: Net-(U2-Pad2) -> K2_2
- U2 pad 22: Net-(U2-Pad22) -> K3_5
- U2 pad 23: Net-(U2-Pad23) -> K2_5
- U2 pad 24: Net-(U2-Pad24) -> K1_6
- U2 pad 25: Net-(U2-Pad25) -> K0_7
- U2 pad 26: Net-(U2-Pad26) -> K2_6
- U2 pad 29: Net-(U2-Pad29) -> K3_6
- U2 pad 3: Net-(U2-Pad3) -> K1_3
- U2 pad 30: Net-(U2-Pad30) -> K4_3
- U2 pad 31: Net-(U2-Pad31) -> K3_7
- U2 pad 32: Net-(U2-Pad32) -> K1_7
- U2 pad 33: Net-(U2-Pad33) -> K2_7
- U2 pad 34: Net-(U2-Pad34) -> K3_8
- U2 pad 35: Net-(U2-Pad35) -> K0_8
- U2 pad 36: Net-(U2-Pad36) -> K1_8
- U2 pad 37: Net-(U2-Pad37) -> K2_8
- U2 pad 38: Net-(U2-Pad38) -> K3_9
- U2 pad 39: Net-(U2-Pad39) -> K4_4
- U2 pad 4: Net-(U2-Pad4) -> K0_4
- U2 pad 40: Net-(U2-Pad40) -> K0_9
- U2 pad 41: Net-(U2-Pad41) -> K1_9
- U2 pad 42: Net-(U2-Pad42) -> K2_9
- U2 pad 43: Net-(U2-Pad43) -> K3_10
- U2 pad 44: Net-(U2-Pad44) -> K4_5
- U2 pad 45: Net-(U2-Pad45) -> K0_10
- U2 pad 46: Net-(U2-Pad46) -> K1_10
- U2 pad 47: Net-(U2-Pad47) -> K2_10
- U2 pad 48: Net-(U2-Pad48) -> K3_11
- U2 pad 5: Net-(U2-Pad5) -> K4_2
- U2 pad 51: Net-(U2-Pad51) -> K4_6
- U2 pad 52: Net-(U2-Pad52) -> K4_7
- U2 pad 53: Net-(U2-Pad53) -> K0_11
- U2 pad 54: Net-(U2-Pad54) -> K1_11
- U2 pad 55: Net-(U2-Pad55) -> K2_11
- U2 pad 56: Net-(U2-Pad56) -> K3_12
- U2 pad 57: Net-(U2-Pad57) -> K0_12
- U2 pad 58: Net-(U2-Pad58) -> K1_12
- U2 pad 59: Net-(U2-Pad59) -> K2_12
- U2 pad 60: Net-(U2-Pad60) -> K3_13
- U2 pad 61: Net-(U2-Pad61) -> K0_13
- U2 pad 62: Net-(U2-Pad62) -> K0_14
- U2 pad 63: Net-(U2-Pad63) -> K1_13
- U2 pad 64: Net-(U2-Pad64) -> K4_8
- U2 pad 7: Net-(U2-Pad7) -> K3_3
- U2 pad 83: Net-(U2-Pad83) -> K0_0
- U2 pad 84: Net-(U2-Pad84) -> K1_0
- U2 pad 85: Net-(U2-Pad85) -> K0_1
- U2 pad 86: Net-(U2-Pad86) -> K2_0
- U2 pad 87: Net-(U2-Pad87) -> K3_0
- U2 pad 88: Net-(U2-Pad88) -> K1_1
- U2 pad 89: Net-(U2-Pad89) -> K0_2
- U2 pad 90: Net-(U2-Pad90) -> K4_0
- U2 pad 91: Net-(U2-Pad91) -> K3_1
- U2 pad 95: Net-(U2-Pad95) -> K2_1
- U2 pad 96: Net-(U2-Pad96) -> K1_2
- U2 pad 97: Net-(U2-Pad97) -> K0_3
- U2 pad 98: Net-(U2-Pad98) -> K4_1
Routing:
- net K4_3: track 0.00 -> 106.0 mm
- net K3_6: track 0.00 -> 75.2 mm
- net K3_7: track 0.00 -> 72.9 mm
- net K2_6: track 0.00 -> 51.2 mm
- net GND: track 0.00 -> 4.54 mm, vias 0 -> 1

Commit message: right switch traces
Connections:
- U2 pad 61: K0_13 -> K4_8
- U2 pad 62: K0_14 -> K1_13
- U2 pad 63: K1_13 -> K0_13
- U2 pad 64: K4_8 -> K0_14
Routing:
- net K4_8: track 0.00 -> 199.6 mm
- net K3_13: track 0.00 -> 176.1 mm
- net K4_7: track 0.00 -> 169.6 mm
- net K3_12: track 0.00 -> 161.9 mm
- net K4_6: track 0.00 -> 151.9 mm
- net K2_12: track 0.00 -> 151.2 mm
- net K1_13: track 0.00 -> 148.6 mm
- net K0_14: track 0.00 -> 141.6 mm
- net K4_5: track 0.00 -> 140.3 mm
- net K0_13: track 0.00 -> 131.5 mm
- net K3_11: track 0.00 -> 126.0 mm
- net K2_11: track 0.00 -> 125.5 mm
- net K1_12: track 0.00 -> 124.3 mm
- net K4_4: track 0.00 -> 117.5 mm
- net K3_10: track 0.00 -> 108.0 mm
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
Commit message: Routed PCB
Parts:
- added J6: Conn_01x03, Connector_PinHeader_2.54mm:PinHeader_1x03_P2.54mm_Vertical, F.Cu at (224.4, -118.1)
- added Ref**: Val**, kobuss-footprint:kobuss_name, F.Cu at (275.7, -97.3)
- added Ref**: Val**, kobuss-footprint:kobuss_name, B.Cu at (275.7, -97.3)
- moved U1 23.6 mm to (246.4, -101.6)
- moved C1 14.5 mm to (248.9, -107.3), turned to 90 degrees
- moved J1 14.0 mm to (14.0, -118.1)
- moved R2 14.0 mm to (6.35, -118.1)
- moved J2 12.7 mm to (25.4, -118.1)
- moved R1 12.7 mm to (20.3, -118.1)
- moved C2 9.79 mm to (240.5, -107.3), turned to 90 degrees
- moved R4 3.24 mm to (244.5, -107.3), turned to -90 degrees
- moved R3 0.63 mm to (246.4, -107.3), turned to -90 degrees
Connections:
- net DM renamed D_N
- net DP renamed D_P
- U2 pad 65: Net-(U2-Pad65) -> ENC_SW
- U2 pad 66: Net-(U2-Pad66) -> ENC_A
- U2 pad 67: Net-(U2-Pad67) -> ENC_B
- U2 pad 68: Net-(U2-Pad68) -> PA9
Routing:
- net +3V3: track 4.10 -> 303.6 mm, vias 1 -> 3
- net K4_0: track 0.00 -> 186.4 mm
- net K3_0: track 0.00 -> 182.8 mm
- net K2_0: track 0.00 -> 161.6 mm
- net K4_1: track 0.00 -> 160.8 mm
- net K3_1: track 0.00 -> 158.8 mm
- net K1_0: track 0.00 -> 152.6 mm
- net I2C_DAT: track 0.00 -> 141.3 mm, vias 0 -> 2
- net K0_0: track 0.00 -> 141.0 mm
- net BOOT: track 0.00 -> 139.2 mm, vias 0 -> 1
- net I2C_CLK: track 0.00 -> 136.3 mm, vias 0 -> 2
- net K4_2: track 0.00 -> 135.8 mm
- net ENC_SW: track 0.00 -> 135.1 mm
- net ENC_A: track 0.00 -> 133.2 mm
- net K2_1: track 0.00 -> 132.9 mm
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- added copper zone on B.Cu, net GND
- added copper zone on F.Cu, net GND
Other:
- board text added: "5V GND PA9"
- board text added: "BOOT"
- board text added: "RESET"
- board text added: "SWDEBUG"
